File: Testa projekts/Jekabs_ilja_Sumo_Test.kicad_pcb (KiCad board)
At the start: 2 copper layers, 138 x 79 mm, 40 parts, among them J1 Conn_01x03, J2 Conn_01x03, J3 Edge_BL, J4 Edge_FR, J5 Conn_01x03, J6 Conn_01x03, J7 Edge_BR, J8 Edge_FL, Q1 Q_Photo, Q2 Q_Photo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

Commit message: Projekta nosaukuma maiņa un ražošanas PCB failu korekcijas
Routing:
- net +5V: track 374.3 -> 373.4 mm
