File: Testa projekts/Infrared_sensors.sch (KiCad schematic (older format))
At the start: 36 parts, among them J1 Conn_01x03, J2 Conn_01x03, J3 Conn_01x03, J4 Conn_01x03, J5 Conn_01x03, J6 Conn_01x03, J7 Conn_01x03, J8 Conn_01x03, Q1 Q_Photo, Q2 Q_Photo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

Commit message: Testa principiālās shēmas pdf sagatave
Other:
- note added: "V_out = 0,4 + 1,9dV\noutput period = 38.3ms ± 9.6ms\nmeasure to output delay = period + 5ms\nexpected reaction time of around 45ms ± 10ms"
- note removed: "V_out = 0,4 + 1,9dV\noutput period = 38.3ms ± 9.6ms\nmeasure to output delay = T + 5ms\nexpected reaction time of around 45ms ± 10ms"
- moved on the sheet: D1, D2, D3, D4, J1, J2, J3, J4, J5, J6, J7, J8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
