File: Testa projekts/Production files/Motherboard/Jekabs_ilja_Sumo_Test_Motherboard.kicad_pcb (KiCad board)
At the start: 2 copper layers, 82 x 79 mm, 16 parts, among them J3 Edge_BL, J4 Edge_FR, J7 Edge_BR, J8 Edge_FL, U1 Proximity_FC, U10 MX1508, U11 DFR0379, U2 Proximity_FR, U3 Proximity_R, U4 Proximity_BR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

Commit message: Projekta nosaukuma maiņa un ražošanas PCB failu korekcijas
Routing:
- net +5V: track 308.3 -> 307.4 mm
- net GND: vias 10 -> 13
Other:
- board size 82 x 79 mm -> 81 x 78 mm
